File: test/test.kicad_pcb (KiCad board)
At the start: 2 copper layers, 3 parts, among them SW1 MX_SW_HS, U1 ProMicro

Commit message: add
Parts:
- removed U1: ProMicro, Keebio-Parts:ArduinoProMicro
- moved D1 82.9 mm to (27.7, 71.7)
- moved SW1 82.9 mm to (31.8, 67.5)
